File: Schematics/HotplateReflowSchematic.brd (EAGLE design)
At the start: 88.6 x 57.1 mm, 39 parts, among them IC1 MAX31855, IC2 REG1117, IC3 REG1117, Q1 8Mhz, U1 LCD-16X2SILK

Commit message: Updating schematic to have automatic switching between USB and DC jack
Parts:
- removed S3: (no value), SparkFun-Electromechanical:SWITCH-SPDT
- added C11: 47u, SparkFun-Passives:0603-CAP
- added IC4: LM358D, linear:SO08
- added R12, R13: 10k, SparkFun-Passives:0603-RES
- added U$5: P-CHANNEL-MOSFET-SOT23-3, GeekAmmo:SOT23-3
Connections:
- new net N$8: R12.2, R13.1
- new net N$9: IC4.1, U$5.1
- net 3V3: now also IC4.2
- net 5VO: now also IC4.8; no longer S3.1
- net DCIN: now also C11.1, IC4.3, R13.2
- net GND: now also C11.2, IC4.4, IC4.5, IC4.6, R12.1
- net VBUS: now also U$5.3; no longer S3.3
- net VIN: now also U$5.2; no longer S3.2
Routing:
- net VIN: track 194.7 -> 253.7 mm, vias 2 -> 1
- net VBUS: track 12.7 -> 45.8 mm
- net 5VO: track 39.8 -> 11.5 mm, vias 2 -> 0
- net 3V3: track 136.4 -> 162.1 mm, vias 3 -> 2
- net DCIN: track 12.7 -> 35.1 mm
- net T-: track 30.5 -> 39.0 mm
- net SCK: track 52.3 -> 43.9 mm, vias 1 -> 0
- net N$9: track 0.00 -> 6.29 mm
- net RIGHT: track 30.1 -> 24.1 mm
- net D+: track 10.8 -> 4.92 mm, vias 2 -> 0
- net N$5: track 11.0 -> 5.13 mm, vias 2 -> 0
- net N$1: track 22.3 -> 17.6 mm
- net A5: track 42.2 -> 37.7 mm
- net SELECT: track 36.0 -> 31.6 mm, vias 2 -> 0
- net RESET: track 58.4 -> 54.5 mm
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Other:
- board text added: "TimmehTimmehReflow ver 1.1"
- board text removed: "JCK"
- board text removed: "USB"
