File: Schematics/HotplateReflowSchematic.sch (EAGLE design)
At the start: 39 parts, among them IC1 MAX31855, IC2 REG1117, IC3 REG1117, Q1 8Mhz, U1 LCD-16X2SILK

Commit message: Updating schematic to have automatic switching between USB and DC jack
Parts:
- removed S3: (no value), SparkFun-Electromechanical:SWITCH-SPDTPTH
- added C11: 47u, SparkFun-Passives:CAP0603-CAP
- added IC4: LM358D, linear:LM358D
- added R12, R13: 10k, SparkFun-Passives:RESISTOR0603-RES
- added U$5: P-CHANNEL-MOSFET-SOT23-3, GeekAmmo:P-CHANNEL-MOSFET-SOT23-3
Connections:
- new net N$8: R12.2, R13.1
- new net N$9: IC4A.OUT, U$5.G
- net 3V3: now also IC4A.-IN
- net 5VO: now also IC4P.V+; no longer S3.O
- net DCIN: now also C11.1, IC4A.+IN, R13.2
- net GND: now also C11.2, IC4B.+IN, IC4B.-IN, IC4P.V-, R12.1
- net VBUS: now also U$5.D; no longer S3.S
- net VIN: now also U$5.S; no longer S3.P
Other:
- moved on the sheet: C10, U$3
Changed lines of the file:
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@@
 <?xml version="1.0" encoding="utf-8"?>
 <!DOCTYPE eagle SYSTEM "eagle.dtd">
-<eagle version="7.5.0">
+<eagle version="7.6.0">
 <drawing>
 <settings>
@@
 <part name="R11" library="SparkFun-Passives" deviceset="RESISTOR" device="0603-RES" value="10k"/>
 <part name="U$4" library="GeekAmmo" deviceset="USB-CON-5PIN" device="-105017-0001"/>
-<part name="S3" library="SparkFun-Electromechanical" deviceset="SWITCH-SPDT" device="PTH"/>
 <part name="S2" library="SparkFun-Electromechanical" deviceset="STANDOFF_ELECTRICAL" device=""/>
 <part name="S4" library="SparkFun-Electromechanical" deviceset="STANDOFF_ELECTRICAL" device=""/>
 <part name="GND16" library="supply1" deviceset="GND" device=""/>
 <part name="GND17" library="supply1" deviceset="GND" device=""/>
+<part name="R12" library="SparkFun-Passives" deviceset="RESISTOR" device="0603-RES" value="10k"/>
+<part name="R13" library="SparkFun-Passives" deviceset="RESISTOR" device="0603-RES" value="10k"/>
+<part name="C11" library="SparkFun-Passives" deviceset="CAP" device="0603-CAP" value="47u"/>
+<part name="GND18" library="SparkFun-Aesthetics" deviceset="GND" device=""/>
+<part name="GND19" library="SparkFun-Aesthetics" deviceset="GND" device=""/>
+<part name="U$5" library="GeekAmmo" deviceset="P-CHANNEL-MOSFET" device="-SOT23-3"/>
+<part name="GND20" library="SparkFun-Aesthetics" deviceset="GND" device=""/>
+<part name="GND21" library="SparkFun-Aesthetics" deviceset="GND" device=""/>
+<part name="IC4" library="linear" deviceset="LM358" device="D"/>
 </parts>
 <sheets>
@@
 <instance part="GND9" gate="1" x="66.04" y="63.5"/>
 <instance part="GND10" gate="1" x="170.18" y="182.88"/>
-<instance part="GND11" gate="1" x="12.7" y="124.46"/>
+<instance part="GND11" gate="1" x="-48.26" y="132.08"/>
 <instance part="GND12" gate="1" x="27.94" y="88.9"/>
 <instance part="C3" gate="G$1" x="7.62" y="101.6"/>
@@
 <instance part="JP1" gate="G$1" x="200.66" y="48.26"/>
 <instance part="S1" gate="G$1" x="170.18" y="190.5" rot="R270"/>
-<instance part="U$3" gate="G$1" x="2.54" y="132.08"/>
+<instance part="U$3" gate="G$1" x="-55.88" y="142.24"/>
 <instance part="IC3" gate="G$1" x="27.94" y="55.88"/>
 <instance part="C8" gate="G$1" x="7.62" y="48.26"/>
@@
 <instance part="GND13" gate="1" x="223.52" y="81.28" rot="R180"/>
 <instance part="JP3" gate="G$1" x="190.5" y="104.14" rot="MR180"/>
-<instance part="C10" gate="G$1" x="83.82" y="139.7"/>
-<instance part="GND14" gate="1" x="83.82" y="134.62"/>
+<instance part="C10" gate="G$1" x="33.02" y="129.54" rot="R180"/>
+<instance part="GND14" gate="1" x="33.02" y="134.62" rot="R180"/>
 <instance part="JP2" gate="G$1" x="-48.26" y="104.14"/>
 <instance part="R6" gate="G$1" x="109.22" y="96.52"/>
@@
 <instance part="R11" gate="G$1" x="208.28" y="63.5"/>
 <instance part="U$4" gate="G$1" x="-2.54" y="172.72"/>
-<instance part="S3" gate="1" x="73.66" y="147.32" rot="R180"/>
 <instance part="S2" gate="G$1" x="-35.56" y="76.2"/>
 <instance part="S4" gate="G$1" x="-35.56" y="60.96"/>
 <instance part="GND16" gate="1" x="-27.94" y="73.66"/>
 <instance part="GND17" gate="1" x="-27.94" y="58.42"/>
+<instance part="R12" gate="G$1" x="-20.32" y="127" rot="R90"/>
+<instance part="R13" gate="G$1" x="-20.32" y="139.7" rot="R90"/>
+<instance part="C11" gate="G$1" x="-35.56" y="139.7"/>
+<instance part="GND18" gate="1" x="-20.32" y="119.38"/>
+<instance part="GND19" gate="1" x="-35.56" y="132.08"/>
+<instance part="U$5" gate="G$1" x="7.62" y="127" smashed="yes" rot="R270">
+<attribute name="VALUE" x="-5.08" y="119.38" size="1.778" layer="96"/>
+<attribute name="NAME" x="5.08" y="129.54" size="1.778" layer="95"/>
+</instance>
+<instance part="GND20" gate="1" x="-15.24" y="195.58"/>
+<instance part="GND21" gate="1" x="-7.62" y="137.16"/>
+<instance part="IC4" gate="A" x="-7.62" y="147.32"/>
+<instance part="IC4" gate="B" x="-7.62" y="203.2"/>
+<instance part="IC4" gate="P" x="-7.62" y="147.32"/>
 </instances>
 <busses>
@@
 </segment>
 <segment>
-<wire x1="68.58" y1="149.86" x2="60.96" y2="149.86" width="0.1524" layer="91"/>
-<label x="60.96" y="152.4" size="1.778" layer="95"/>
-<pinref part="S3" gate="1" pin="S"/>
+<pinref part="U$5" gate="G$1" pin="D"/>
+<wire x1="0" y1="124.46" x2="-7.62" y2="124.46" width="0.1524" layer="91"/>
+<label x="-7.62" y="124.46" size="1.778" layer="95"/>
 </segment>
 </net>
@@
 <pinref part="U$3" gate="G$1" pin="RING_SW"/>
 <pinref part="GND11" gate="1" pin="GND"/>
-<wire x1="7.62" y1="132.08" x2="12.7" y2="132.08" width="0.1524" layer="91"/>
-<wire x1="12.7" y1="132.08" x2="12.7" y2="129.54" width="0.1524" layer="91"/>
+<wire x1="-50.8" y1="142.24" x2="-48.26" y2="142.24" width="0.1524" layer="91"/>
+<wire x1="-48.26" y1="142.24" x2="-48.26" y2="139.7" width="0.1524" layer="91"/>
 <pinref part="U$3" gate="G$1" pin="RING"/>
-<wire x1="12.7" y1="129.54" x2="12.7" y2="127" width="0.1524" layer="91"/>
-<wire x1="7.62" y1="129.54" x2="12.7" y2="129.54" width="0.1524" layer="91"/>
-<junction x="12.7" y="129.54"/>
+<wire x1="-48.26" y1="139.7" x2="-48.26" y2="134.62" width="0.1524" layer="91"/>
+<wire x1="-50.8" y1="139.7" x2="-48.26" y2="139.7" width="0.1524" layer="91"/>
+<junction x="-48.26" y="139.7"/>
 </segment>
 <segment>
@@
 <pinref part="GND17" gate="1" pin="GND"/>
 </segment>
+<segment>
+<pinref part="R12" gate="G$1" pin="1"/>
+<pinref part="GND18" gate="1" pin="GND"/>
+</segment>
+<segment>
+<pinref part="C11" gate="G$1" pin="2"/>
+<pinref part="GND19" gate="1" pin="GND"/>
+<wire x1="-35.56" y1="137.16" x2="-35.56" y2="134.62" width="0.1524" layer="91"/>
+</segment>
+<segment>
+<wire x1="-15.24" y1="205.74" x2="-15.24" y2="200.66" width="0.1524" layer="91"/>
+<pinref part="GND20" gate="1" pin="GND"/>
+<pinref part="IC4" gate="B" pin="-IN"/>
+<wire x1="-15.24" y1="200.66" x2="-15.24" y2="198.12" width="0.1524" layer="91"/>
+<junction x="-15.24" y="200.66"/>
+<pinref part="IC4" gate="B" pin="+IN"/>
+</segment>
+<segment>
+<pinref part="GND21" gate="1" pin="GND"/>
+<pinref part="IC4" gate="P" pin="V-"/>
+</segment>
 </net>
 <net name="N$5" class="0">
@@
 <label x="-35.56" y="111.76" size="1.778" layer="95"/>
 </segment>
+<segment>
+<label x="-15.24" y="139.7" size="1.778" layer="95"/>
+<pinref part="IC4" gate="A" pin="-IN"/>
+<wire x1="-15.24" y1="144.78" x2="-15.24" y2="139.7" width="0.1524" layer="91"/>
+</segment>
 </net>
 <net name="XTAL2" class="0">
@@
 </segment>
 <segment>
-<wire x1="76.2" y1="147.32" x2="83.82" y2="147.32" width="0.1524" layer="91"/>
-<label x="78.74" y="147.32" size="1.778" layer="95"/>
 <pinref part="C10" gate="G$1" pin="1"/>
-<wire x1="83.82" y1="147.32" x2="83.82" y2="144.78" width="0.1524" layer="91"/>
-<pinref part="S3" gate="1" pin="P"/>
+<wire x1="15.24" y1="124.46" x2="33.02" y2="124.46" width="0.1524" layer="91"/>
+<pinref part="U$5" gate="G$1" pin="S"/>
+<label x="20.32" y="132.08" size="1.778" layer="95"/>
 </segment>
 <segment>
@@
 <segment>
 <pinref part="U$3" gate="G$1" pin="TIP"/>
-<wire x1="7.62" y1="134.62" x2="15.24" y2="134.62" width="0.1524" layer="91"/>
-<label x="17.78" y="134.62" size="1.778" layer="95"/>
+<label x="-45.72" y="147.32" size="1.778" layer="95"/>
+<pinref part="C11" gate="G$1" pin="1"/>
+<wire x1="-35.56" y1="144.78" x2="-50.8" y2="144.78" width="0.1524" layer="91"/>
+<pinref part="R13" gate="G$1" pin="2"/>
+<wire x1="-35.56" y1="144.78" x2="-20.32" y2="144.78" width="0.1524" layer="91"/>
+<junction x="-35.56" y="144.78"/>
+<wire x1="-12.7" y1="149.86" x2="-15.24" y2="149.86" width="0.1524" layer="91"/>
+<wire x1="-15.24" y1="149.86" x2="-20.32" y2="149.86" width="0.1524" layer="91"/>
+<wire x1="-20.32" y1="149.86" x2="-20.32" y2="144.78" width="0.1524" layer="91"/>
+<junction x="-20.32" y="144.78"/>
+<pinref part="IC4" gate="A" pin="+IN"/>
+<junction x="-15.24" y="149.86"/>
 </segment>
 <segment>
@@
 </segment>
 <segment>
-<wire x1="68.58" y1="144.78" x2="60.96" y2="144.78" width="0.1524" layer="91"/>
-<label x="58.42" y="144.78" size="1.778" layer="95"/>
-<pinref part="S3" gate="1" pin="O"/>
+<wire x1="-7.62" y1="154.94" x2="-15.24" y2="154.94" width="0.1524" layer="91"/>
+<wire x1="-15.24" y1="154.94" x2="-15.24" y2="157.48" width="0.1524" layer="91"/>
+<label x="-17.78" y="157.48" size="1.778" layer="95"/>
+<pinref part="IC4" gate="P" pin="V+"/>
 </segment>
 </net>
@@
 </segment>
 </net>
+<net name="N$8" class="0">
+<segment>
+<pinref part="R12" gate="G$1" pin="2"/>
+<pinref part="R13" gate="G$1" pin="1"/>
+<wire x1="-20.32" y1="134.62" x2="-20.32" y2="132.08" width="0.1524" layer="91"/>
+</segment>
+</net>
+<net name="N$9" class="0">
+<segment>
+<pinref part="U$5" gate="G$1" pin="G"/>
+<wire x1="10.16" y1="132.08" x2="10.16" y2="147.32" width="0.1524" layer="91"/>
+<wire x1="10.16" y1="147.32" x2="0" y2="147.32" width="0.1524" layer="91"/>
+<pinref part="IC4" gate="A" pin="OUT"/>
+</segment>
+</net>
